File: pcb/single/single.sch (KiCad schematic (older format))
At the start: 27 parts, among them J1 USB_A, J10 USB_A, J2 Barrel_Jack_Switch_DC10B, J3 Barrel_Jack_Switch_DC10B, J4 Barrel_Jack_Switch_DC10B, J5 Barrel_Jack_Switch_DC10B, J6 Barrel_Jack_Switch_DC10B, J7 USB_A, J8 USB_A, J9 USB_A, U1_12V1 i6A4W010A033V-001-R, U1_5V1 i6A4W010A033V-001-R

Commit message: As ordered
Parts:
- removed F2: Fuse, box_power:Fuseholder_Cylinder-5x20mm_646_series_22.6_1.5, symbol Device:Fuse
- added D1: Zener_18V, Diode_THT:D_DO-35_SOD27_P7.62mm_Horizontal, symbol Device:D_Zener
- added H1, H2, H3, H4: MountingHole, MountingHole:MountingHole_3.2mm_M3, symbol Mechanical:MountingHole
- added Q1: Q_PMOS_GDS, Package_TO_SOT_THT:TO-220-3_Vertical, symbol Device:Q_PMOS_GDS
- added R1: 300R, Resistor_THT:R_Axial_DIN0207_L6.3mm_D2.5mm_P10.16mm_Horizontal, symbol Device:R
- added TP_12V1, TP_24V1, TP_5V1, TP_GND1: TestPoint, TestPoint:TestPoint_Pad_D4.0mm, symbol Connector:TestPoint
- USB1: renamed from J1; value USB_A -> USB A
- USB2: renamed from J7; value USB_A -> USB A
- USB3: renamed from J8; value USB_A -> USB A
- USB4: renamed from J9; value USB_A -> USB A
- USB5: renamed from J10; value USB_A -> USB A
- renumbered CIN_5V1 to C1, CO2_5V1 to C2, CO1_5V1 to C3, CIN_12V1 to C4, CO2_12V1 to C5, CO1_12V1 to C6, U1_12V1 to Convert_12V1, U1_5V1 to Convert_5V1, J2 to DC1, J3 to DC2, J4 to DC3, J5 to DC4, J6 to DC5, JIN_24V+1 to IN_24V+1, JOUT_24V-1 to IN_24V-1, JOUT_12V1 to OUT_12V1, JOUT_5V1 to OUT_5V1, RUP_5V1 to R2, RUP_12V1 to R3
Connections:
- net 5V_GND is gone; now on net GND: C2.2, C3.2, Convert_5V1.4 (Vout(-)), OUT_5V1.2 (Pin_2), R2.1, USB1.4 (GND), USB1.5 (Shield), USB2.4 (GND), USB2.5 (Shield), USB3.4 (GND), USB3.5 (Shield), USB4.4 (GND), USB4.5 (Shield), USB5.4 (GND), USB5.5 (Shield)
- net GND_12V is gone; now on net GND: C5.2, C6.2, Convert_12V1.4 (Vout(-)), DC1.3, DC2.3, DC3.3, DC4.3, DC5.3, FAN_12V1.2 (Pin_2), OUT_12V1.2 (Pin_2), R3.1
- net 12V: now also TP_12V1.1
- net 24V: now also C1.1, C4.1, Convert_12V1.1 (Vin(+)), Convert_5V1.1 (Vin(+)), D1.1 (K), Q1.3 (S), TP_24V1.1; no longer F1.2, IN_24V+1.1 (Pin_1), IN_24V+1.2 (Pin_2)
- net 5V: now also TP_5V1.1
- net GND: now also R1.2, TP_GND1.1
- new net: F1.2, IN_24V+1.1 (Pin_1), IN_24V+1.2 (Pin_2)
- new net: F1.1, Q1.2 (D)
- new net: D1.2 (A), Q1.1 (G), R1.1
Other:
- moved on the sheet: C1, C2, C3, Convert_5V1, F1, IN_24V+1, IN_24V-1, OUT_5V1, R2, USB1, USB2, USB3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
